File: Kicad/Bil v 1,0/Bil v 1,0.kicad_pcb (KiCad board)
At the start: 4 copper layers, 100 x 75 mm, 15 parts, among them J1 Analog, J2 Digital, J3 Lidar_sensor_adafruit_VL53L0X, J4 Lidar_sensor_adafruit_VL53L0X, J6 Lidar_sensor_adafruit_VL53L0X, M1 Motor_DC, M2 Motor_Servo, M4 Motor_DC, SW2 power switch

Commit message: 1.4.1 updated silkscreens
updated silkscreens with names of modules
Parts:
- Arduino Nano: renamed from J1
- Lidar Front: renamed from J4
- Lidar L: renamed from J3
- Lidar R: renamed from J6
- Moror controller: renamed from U1
- renumbered BT1 to Battery, U2 to DC-DC, J2 to ESP32, M4 to M2, M2 to Servo
Other:
- board text added: "Ludvig August Mai David"
